Commit message: acml implemented and tested. Final commit

File: catkin_ws/src/my_robot/urdf/my_robot.xacro (robot description, xacro)
@@ -58,5 +58,5 @@
   <link name = 'right_wheel'>
 	  <visual name = 'right_wheel_visual'>
-		  <origin xyz="0 0.15 0" rpy = "0 1.5707 1.5707"/>
+		  <origin xyz="0 0 0" rpy = "0 1.5707 1.5707"/>
       <geometry>
         <cylinder radius = '0.1' length = '0.05'/>
@@ -64,5 +64,5 @@
 	  </visual>
     <collision name = 'right_wheel_collision'>
-		  <origin xyz="0 0.15 0" rpy = "0 1.5707 1.5707"/>
+		  <origin xyz="0 0 0" rpy = "0 1.5707 1.5707"/>
       <geometry>
         <cylinder radius = '0.1' length = '0.05'/>
@@ -80,5 +80,5 @@
   </link>
   <joint name = "right_wheel_hinge" type = "continuous">
-    <origin xyz = "0 0 0" rpy = "0 0 0" />
+    <origin xyz = "0 -0.15 0" rpy = "0 0 0" />
     <child link = "right_wheel"/>
     <parent link = "chassis"/>
@@ -89,5 +89,5 @@
   <link name = 'left_wheel'>
 	  <visual name = 'left_wheel_visual'>
-		  <origin xyz="0 -0.15 0" rpy = "0 1.5707 1.5707"/>
+		  <origin xyz="0 0 0" rpy = "0 1.5707 1.5707"/>
       <geometry>
         <cylinder radius = '0.1' length = '0.05'/>
@@ -95,5 +95,5 @@
 	  </visual>
     <collision name = 'left_wheel_collision'>
-		  <origin xyz="0 -0.15 0" rpy = "0 1.5707 1.5707"/>
+		  <origin xyz="0 0 0" rpy = "0 1.5707 1.5707"/>
       <geometry>
         <cylinder radius = '0.1' length = '0.05'/>
@@ -111,5 +111,5 @@
   </link>
   <joint name = "left_wheel_hinge" type = "continuous">
-    <origin xyz = "0 0 0" rpy = "0 0 0" />
+    <origin xyz = "0 0.15 0" rpy = "0 0 0" />
     <child link = "left_wheel"/>
     <parent link = "chassis"/>
@@ -148,5 +148,5 @@
   <link name = 'hokuyo'>
 	  <visual name = 'hokuyo_visual'>
-		  <origin xyz="0.15 0 0.1" rpy = "0 0 0"/>
+		  <origin xyz="0.0 0.0 0.0" rpy = "0 0 0"/>
       <geometry>
         <mesh filename = "package://my_robot/meshes/hokuyo.dae"/>
@@ -154,7 +154,7 @@
 	  </visual>
     <collision name = 'hokuyo_collision'>
-		  <origin xyz="0.2 0 0" rpy = "0 0 0"/>
+		  <origin xyz="0.0 0 0" rpy = "0 0 0"/>
       <geometry>
-        <box size = "0.05 0.05 0.1"/>
+        <box size = "0.1 0.1 0.1"/>
       </geometry>
 	  </collision>
@@ -169,5 +169,5 @@
   </link>
   <joint name = "hokuyo_joint" type = "fixed">
-    <origin xyz = "0 0 0" rpy = "0 0 0" />
+    <origin xyz = "0.15 0.0 0.1" rpy = "0 0 0" />
     <child link = "hokuyo"/>
     <parent link = "chassis"/>
